File: nimh_charger.sch (KiCad schematic (older format))
At the start: 28 parts, among them J1 USB_B_Micro, J2 Bat +, J3 Bat -, Q1 Q_PMOS_DGS, Q2 2N2219, Q3 Q_PMOS_DGS, Q4 Q_PMOS_DGS, U1 LM317L_TO92, U2 LM339

Commit message: Placed parts on board file. Need to verify the bom before doing more layout
Parts:
- removed J1: USB_B_Micro, Connector_USB:USB_Micro-B_Amphenol_10103594-0001LF_Horizontal, symbol Connector:USB_B_Micro
- added J1: USB_B_Mini, symbol Connector:USB_B_Mini
- Q1, Q3, Q4: footprint (none) -> Package_TO_SOT_SMD:SOT-23
- U2: footprint (none) -> Package_SO:SOIC-14_3.9x8.7mm_P1.27mm
Connections:
- net +5V: now also J1.1 (VBUS)
- net GNDREF: now also J1.5 (GND)
Changed lines of the file:
@@
 F 0 "Q1" V 3792 1450 50  0000 C CNN
 F 1 "Q_PMOS_DGS" V 3701 1450 50  0000 C CNN
-F 2 "" H 3650 1550 50  0001 C CNN
+F 2 "Package_TO_SOT_SMD:SOT-23" H 3650 1550 50  0001 C CNN
 F 3 "~" H 3450 1450 50  0001 C CNN
 	1    3450 1450
@@
 F 0 "Q3" V 7042 1450 50  0000 C CNN
 F 1 "Q_PMOS_DGS" V 6951 1450 50  0000 C CNN
-F 2 "" H 6900 1550 50  0001 C CNN
+F 2 "Package_TO_SOT_SMD:SOT-23" H 6900 1550 50  0001 C CNN
 F 3 "~" H 6700 1450 50  0001 C CNN
 	1    6700 1450
@@
 F 0 "U2" H 6708 2546 50  0000 L CNN
 F 1 "LM339" H 6708 2455 50  0000 L CNN
-F 2 "" H 6700 2600 50  0001 C CNN
+F 2 "Package_SO:SOIC-14_3.9x8.7mm_P1.27mm" H 6700 2600 50  0001 C CNN
 F 3 "https://www.st.com/resource/en/datasheet/lm139.pdf" H 6800 2700 50  0001 C CNN
 	5    6750 2500
@@
 F 0 "U2" H 5700 2867 50  0000 C CNN
 F 1 "LM339" H 5700 2776 50  0000 C CNN
-F 2 "" H 5650 2600 50  0001 C CNN
+F 2 "Package_SO:SOIC-14_3.9x8.7mm_P1.27mm" H 5650 2600 50  0001 C CNN
 F 3 "https://www.st.com/resource/en/datasheet/lm139.pdf" H 5750 2700 50  0001 C CNN
 	1    5700 2500
@@
 F 0 "U2" H 5750 3767 50  0000 C CNN
 F 1 "LM339" H 5750 3676 50  0000 C CNN
-F 2 "" H 5700 3500 50  0001 C CNN
+F 2 "Package_SO:SOIC-14_3.9x8.7mm_P1.27mm" H 5700 3500 50  0001 C CNN
 F 3 "https://www.st.com/resource/en/datasheet/lm139.pdf" H 5800 3600 50  0001 C CNN
 	2    5750 3400
@@
 F 0 "Q4" V 7992 1450 50  0000 C CNN
 F 1 "Q_PMOS_DGS" V 7901 1450 50  0000 C CNN
-F 2 "" H 7850 1550 50  0001 C CNN
+F 2 "Package_TO_SOT_SMD:SOT-23" H 7850 1550 50  0001 C CNN
 F 3 "~" H 7650 1450 50  0001 C CNN
 	1    7650 1450
@@
 Wire Wire Line
 	5100 1350 5700 1350
-$Comp
-L Connector:USB_B_Micro J1
-U 1 1 604FD26C
+Wire Wire Line
+	2150 1350 2400 1350
+Connection ~ 2400 1350
+Wire Wire Line
+	2400 1350 2650 1350
+Wire Wire Line
+	1850 1950 2350 1950
+Wire Wire Line
+	2350 1950 2350 2250
+$Comp
+L Connector:USB_B_Mini J1
+U 1 1 60AA5CAE
 P 1850 1550
 F 0 "J1" H 1907 2017 50  0000 C CNN
-F 1 "USB_B_Micro" H 1907 1926 50  0000 C CNN
-F 2 "Connector_USB:USB_Micro-B_Amphenol_10103594-0001LF_Horizontal" H 2000 1500 50  0001 C CNN
+F 1 "USB_B_Mini" H 1907 1926 50  0000 C CNN
+F 2 "" H 2000 1500 50  0001 C CNN
 F 3 "~" H 2000 1500 50  0001 C CNN
 	1    1850 1550
 	1    0    0    -1
 $EndComp
-Wire Wire Line
-	2150 1350 2400 1350
-Connection ~ 2400 1350
-Wire Wire Line
-	2400 1350 2650 1350
-Wire Wire Line
-	1850 1950 2350 1950
-Wire Wire Line
-	2350 1950 2350 2250
 $EndSCHEMATC

Commit message: Sorted out some footprints. Working on layout and placement.
Parts:
- removed U1: LM317L_TO92, Package_TO_SOT_THT:TO-92_Inline, symbol Regulator_Linear:LM317L_TO92
- added U1: LM317_3PinPackage, Package_TO_SOT_SMD:SOT-223-3_TabPin2, symbol Regulator_Linear:LM317_3PinPackage
- J1: footprint (none) -> Connector_USB:USB_Mini-B_Lumberg_2486_01_Horizontal
- Q2: footprint Package_TO_SOT_THT:TO-39-3 -> Package_TO_SOT_SMD:SOT-23
Connections:
- net at Q1.3 (S), R3.2: now also U1.3 (VI)
- net at D3.2 (A), Q4.3 (S), R12.1: now also U1.1 (ADJ)
- net at R8.2: now also U1.2 (VO)
Changed lines of the file:
@@
 Wire Wire Line
 	4000 2150 4000 2250
-$Comp
-L Regulator_Linear:LM317L_TO92 U1
-U 1 1 604752C8
-P 4800 1350
-F 0 "U1" H 4800 1592 50  0000 C CNN
-F 1 "LM317L_TO92" H 4800 1501 50  0000 C CNN
-F 2 "Package_TO_SOT_THT:TO-92_Inline" H 4800 1575 50  0001 C CIN
-F 3 "http://www.ti.com/lit/ds/snvs775k/snvs775k.pdf" H 4800 1350 50  0001 C CNN
-	1    4800 1350
-	1    0    0    -1
-$EndComp
 Wire Wire Line
 	4000 1350 4500 1350
@@
 F 0 "Q2" H 3690 3146 50  0000 L CNN
 F 1 "2N2219" H 3690 3055 50  0000 L CNN
-F 2 "Package_TO_SOT_THT:TO-39-3" H 3700 3025 50  0001 L CIN
+F 2 "Package_TO_SOT_SMD:SOT-23" H 3700 3025 50  0001 L CIN
 F 3 "http://www.onsemi.com/pub_link/Collateral/2N2219-D.PDF" H 3500 3100 50  0001 L CNN
 	1    3500 3100
@@
 F 0 "J1" H 1907 2017 50  0000 C CNN
 F 1 "USB_B_Mini" H 1907 1926 50  0000 C CNN
-F 2 "" H 2000 1500 50  0001 C CNN
+F 2 "Connector_USB:USB_Mini-B_Lumberg_2486_01_Horizontal" H 2000 1500 50  0001 C CNN
 F 3 "~" H 2000 1500 50  0001 C CNN
 	1    1850 1550
 	1    0    0    -1
 $EndComp
+$Comp
+L Regulator_Linear:LM317_3PinPackage U1
+U 1 1 60B707CA
+P 4800 1350
+F 0 "U1" H 4800 1592 50  0000 C CNN
+F 1 "LM317_3PinPackage" H 4800 1501 50  0000 C CNN
+F 2 "Package_TO_SOT_SMD:SOT-223-3_TabPin2" H 4800 1600 50  0001 C CIN
+F 3 "http://www.ti.com/lit/ds/symlink/lm317.pdf" H 4800 1350 50  0001 C CNN
+	1    4800 1350
+	1    0    0    -1
+$EndComp

Commit message: Added some mounting holes
Parts:
- added H1, H2: MountingHole, MountingHole:MountingHole_3mm, symbol Mechanical:MountingHole
Changed lines of the file:
@@
+	1    0    0    -1
+$EndComp
+$Comp
+L Mechanical:MountingHole H1
+U 1 1 610F8324
+P 850 750
+F 0 "H1" H 950 796 50  0000 L CNN
+F 1 "MountingHole" H 950 705 50  0000 L CNN
+F 2 "MountingHole:MountingHole_3mm" H 850 750 50  0001 C CNN
+F 3 "~" H 850 750 50  0001 C CNN
+	1    850  750
+	1    0    0    -1
+$EndComp
+$Comp
+L Mechanical:MountingHole H2
+U 1 1 610F90F1
+P 850 950
+F 0 "H2" H 950 996 50  0000 L CNN
+F 1 "MountingHole" H 950 905 50  0000 L CNN
+F 2 "MountingHole:MountingHole_3mm" H 850 950 50  0001 C CNN
+F 3 "~" H 850 950 50  0001 C CNN
+	1    850  950
 	1    0    0    -1
 $EndComp
